File: PCB/Motherboard.brd (EAGLE design)
At the start: 100.3 x 69.8 mm, 30 parts, among them IC1 7805TV, IC2 NE555, Q1 BS250

Commit message: Renamed some signals
Connections:
- net N$22 renamed A0
- net N$23 renamed A1
- net N$24 renamed A2
- net N$25 renamed A3
- net N$4 renamed S
- net N$5 renamed G
Changed lines of the file:
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@@
 <wire x1="36.83" y1="57.15" x2="33.02" y2="53.34" width="0.4064" layer="16"/>
 </signal>
-<signal name="N$4">
+<signal name="S">
 <contactref element="9V" pad="1"/>
 <contactref element="Q1" pad="S"/>
@@
 <wire x1="96.52" y1="22.86" x2="95.25" y2="22.86" width="0.4064" layer="16"/>
 </signal>
-<signal name="N$5">
+<signal name="G">
 <contactref element="IC1" pad="3"/>
 <contactref element="C2" pad="+"/>
@@
 <wire x1="21.51" y1="56.388" x2="21.51" y2="66.06" width="1.016" layer="16"/>
 </signal>
-<signal name="N$22">
+<signal name="A0">
 <contactref element="ARDUINO_NANO1" pad="4"/>
 <contactref element="X6" pad="1"/>
@@
 <wire x1="88.9" y1="51.181" x2="88.9" y2="64.65" width="0.4064" layer="16"/>
 </signal>
-<signal name="N$23">
+<signal name="A1">
 <contactref element="ARDUINO_NANO1" pad="5"/>
 <contactref element="X6" pad="2"/>
@@
 <wire x1="85.344" y1="63.206" x2="82.51" y2="66.04" width="0.4064" layer="16"/>
 </signal>
-<signal name="N$24">
+<signal name="A2">
 <contactref element="ARDUINO_NANO1" pad="6"/>
 <contactref element="X6" pad="3"/>
@@
 <wire x1="82.804" y1="59.436" x2="77.51" y2="64.73" width="0.4064" layer="16"/>
 </signal>
-<signal name="N$25">
+<signal name="A3">
 <contactref element="ARDUINO_NANO1" pad="7"/>
 <contactref element="X6" pad="4"/>
